File: kicad/cosmac_toy_v2/cosmac_toy_v2.kicad_pcb (KiCad board)
At the start: 2 copper layers, 72 x 95 mm, 61 parts, among them J1 Conn_01x20, J2 Conn_01x20, J3 Barrel_Jack_Switch, SW1 D0, SW10 CLEAR, SW11 STB SW, SW12 DMA-IN, SW13 R/W SW, SW2 D1, SW3 D2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

Commit message: Added KiCad project Rev.0.3
Parts:
- removed the R5 at (87.0, 62.6)
- removed the R6 at (87.0, 59.4)
- removed the R7 at (47.6, 101.3)
- added J4: USB-C Power, A295-CTRPB-1:A295-CTRPB-1, F.Cu at (89.5, 147.7)
- added RN5: RN100K-4, Resistor_THT:R_Array_SIP5, F.Cu at (40.0, 101.3)
- R1, R3: value 22k -> 100k
- R5: renamed from R8; value 22k -> 100k
- R6: renamed from R9; value 22k -> 100k
- R7: renamed from R10; value 22k -> 100k
- R8: renamed from R11; value 22k -> 100k
- RN1: value RN22K-8 -> RN100K-8
- RN2: value RN22K-4 -> RN100K-4
- RN4: value RN6.8K-8 -> RN10K-8
- moved RN4 20.3 mm to (43.8, 87.4), turned to 0 degrees
- moved D4 11.5 mm to (75.6, 133.7), turned to 0 degrees
- moved D2 7.62 mm to (83.8, 59.4), turned to 180 degrees
- moved D3 7.62 mm to (83.8, 62.2), turned to 180 degrees
- moved J3 4.45 mm to (79.1, 137.3)
- moved RN1 3.18 mm to (54.0, 101.3)
- moved R4 1.42 mm to (77.5, 129.3)
- moved LED1 1.27 mm to (92.7, 81.7)
- moved LED2 1.27 mm to (85.7, 81.7)
- moved LED3 1.27 mm to (78.7, 81.7)
- moved LED4 1.27 mm to (71.8, 81.7)
- moved SW3 1.27 mm to (80.0, 92.5)
- moved SW1 1.27 mm to (94.0, 92.5)
- moved SW2 1.27 mm to (87.0, 92.5)
- moved SW4 1.27 mm to (73.0, 92.5)
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Connections:
- J2 pad 4: VDD -> /~{DMAOUT}
- SW1 pad 2: Net-(RN4-R1) -> Net-(RN4-R8)
- SW2 pad 2: Net-(RN4-R2) -> Net-(RN4-R7)
- SW3 pad 2: Net-(RN4-R3) -> Net-(RN4-R6)
- SW4 pad 2: Net-(RN4-R4) -> Net-(RN4-R5)
- SW5 pad 2: Net-(RN4-R5) -> Net-(RN4-R4)
- SW6 pad 2: Net-(RN4-R6) -> Net-(RN4-R3)
- SW7 pad 2: Net-(RN4-R7) -> Net-(RN4-R2)
- SW8 pad 2: Net-(RN4-R8) -> Net-(RN4-R1)
- U1 pad 37: VDD -> /~{DMAOUT}
Routing:
- net Net-(RN4-R1): track 34.6 -> 8.67 mm
- net Net-(RN4-R8): track 8.51 -> 33.0 mm
- net Net-(RN4-R2): track 29.8 -> 8.45 mm
- net /D3: track 97.5 -> 76.6 mm
- net Net-(RN4-R7): track 9.50 -> 28.6 mm
- net VDD: track 286.1 -> 268.0 mm
- net /~{CLEAR}: track 148.0 -> 165.1 mm, vias 1 -> 2
- net Net-(RN4-R3): track 25.4 -> 10.3 mm
- net /~{WAIT}: track 113.8 -> 100.2 mm
- net Net-(D2-K): track 25.8 -> 13.4 mm
- net Net-(RN4-R6): track 12.0 -> 24.1 mm
- net /~{DMAOUT}: track 0.00 -> 7.51 mm
- net /SC1: track 116.5 -> 109.3 mm, vias 1 -> 2
- net Net-(RN4-R4): track 20.9 -> 14.0 mm
- net Net-(D3-K): track 12.3 -> 6.64 mm
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Other:
- board text added: "+5V"
- board text added: "Rev.0.3 2024-12-12 @kanpapa"
- board text removed: "5V"
- board text removed: "Rev.0.2 2024-11-27 @kanpapa"
