File: kicad/cosmac_toy_v2/cosmac_toy_v2.kicad_sch (KiCad schematic)
At the start: 57 parts, among them J1 Conn_01x20, J2 Conn_01x20, J3 Barrel_Jack_Switch, SW1 D0, SW10 CLEAR, SW11 STB SW, SW12 DMA-IN, SW13 R/W SW, SW2 D1, SW3 D2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

Commit message: Added KiCad project Rev.0.3
Parts:
- removed R5, R6, R7: 100k, Resistor_THT:R_Axial_DIN0207_L6.3mm_D2.5mm_P7.62mm_Horizontal, symbol Device:R
- added J4: USB-C Power, A295-CTRPB-1:A295-CTRPB-1, symbol Connector_Generic:Conn_01x03
- added RN5: RN100K-4, Resistor_THT:R_Array_SIP5, symbol Device:R_Network04
- renumbered R8 to R5, R9 to R6, R10 to R7, R11 to R8
Connections:
- net GND: now also J4.2 (Pin_2), J4.3 (Pin_3)
- net VDD: now also J4.1 (Pin_1), RN5.1 (common); no longer J2.4 (Pin_4), U1.37 (~{DMA_OUT})
- net ~{CLEAR}: now also RN5.3 (R2)
- net ~{INT}: now also RN5.5 (R4)
- net ~{WAIT}: now also RN5.2 (R1)
- net at SW5.2 (B): now also RN4.5 (R4); no longer RN4.6 (R5)
- net at SW3.2 (B): now also RN4.7 (R6); no longer RN4.4 (R3)
- net at SW4.2 (B): now also RN4.6 (R5); no longer RN4.5 (R4)
- net at RN4.2 (R1): now also SW8.2 (B); no longer SW1.2 (B)
- net at SW6.2 (B): now also RN4.4 (R3); no longer RN4.7 (R6)
- net at RN4.3 (R2): now also SW7.2 (B); no longer SW2.2 (B)
- net at RN4.8 (R7): now also SW2.2 (B); no longer SW7.2 (B)
- net at RN4.9 (R8): now also SW1.2 (B); no longer SW8.2 (B)
- new net ~{DMAOUT}: J2.4 (Pin_4), RN5.4 (R3), U1.37 (~{DMA_OUT})
